File: project-files/qsb/RGB Encoder Switcher QSB v1p2.brd (EAGLE design)
At the start: 15.2 x 49.5 mm, 11 parts

Commit message: Add files via upload
Routing:
- net LOGO: track 0.00 -> 22.6 mm
- net N$17: track 8.00 -> 0.00 mm
- net N$16: track 6.48 -> 0.00 mm
- net N$18: track 5.16 -> 0.00 mm
- net N$23: track 3.00 -> 0.00 mm
- net GND: track 7.37 -> 5.79 mm
- net Z80_CLK_IN: track 18.8 -> 18.9 mm, vias 0 -> 1
Changed lines of the file:
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@@
 </classes>
 <designrules name="oshpark-2layer *">
-<description language="en">&lt;b&gt;OSH Park Design Rules&lt;/b&gt;
-&lt;p&gt;
-Please make sure your boards conform to these design rules.
-&lt;/p&gt;
-&lt;p&gt;
-Note, that not all DRC settings must be set by the manufacturer. Several can be adjusted for the design, including those listed on our docs page here.
-&lt;a href=&quot;http://docs.oshpark.com/design-tools/eagle/design-rules-files/&quot;&gt;Adjustable Settings&lt;/a&gt;
-&lt;/p&gt;</description>
+<description language="en">&lt;b&gt;Consoles Unleashed Design Rules&lt;/b&gt;</description>
 <param name="layerSetup" value="(1*16)"/>
 <param name="mtCopper" value="0.035559375mm 0.0356mm 0.0356mm 0.0356mm 0.0356mm 0.0356mm 0.0356mm 0.0356mm 0.0356mm 0.0356mm 0.0356mm 0.0356mm 0.0356mm 0.0356mm 0.0356mm 0.035559375mm"/>
@@
 <contactref element="C1" pad="1"/>
 <contactref element="C2" pad="2"/>
-<wire x1="11.01" y1="22.86" x2="10.83369375" y2="22.86" width="0.508" layer="1"/>
 <wire x1="11.01" y1="22.86" x2="10.85125" y2="22.70125" width="0.508" layer="1"/>
 <wire x1="10.85125" y1="22.70125" x2="10.85125" y2="21.54645" width="0.508" layer="1"/>
@@
 <contactref element="INVERTER" pad="2"/>
 <contactref element="MULTIPLEXER" pad="1"/>
-<wire x1="8.9154" y1="25.7302" x2="8.6654" y2="25.7302" width="0.508" layer="1"/>
 <wire x1="1.905" y1="3.81" x2="2.69875" y2="4.60375" width="0.8" layer="1"/>
 <via x="3.095625" y="5.000625" extent="1-16" drill="0.4" diameter="0.8"/>
@@
 <wire x1="14.76375" y1="34.925" x2="13.335" y2="35.56" width="0.4064" layer="1" curve="20"/>
 <wire x1="6.3246" y1="28.09875" x2="6.0071" y2="27.78125" width="0.1524" layer="1"/>
-<wire x1="6.0071" y1="27.78125" x2="5.794375" y2="27.78125" width="0.1524" layer="1"/>
-<wire x1="6.3246" y1="28.09875" x2="6.6421" y2="27.78125" width="0.1524" layer="1"/>
-<wire x1="6.6421" y1="27.78125" x2="6.82625" y2="27.78125" width="0.1524" layer="1"/>
+<wire x1="6.6421" y1="27.78125" x2="6.3246" y2="28.09875" width="0.1524" layer="1"/>
+<via x="15.24" y="35.56" extent="1-16" drill="1" diameter="2"/>
+<wire x1="6.3246" y1="27.6098" x2="6.3246" y2="27.78125" width="0.1524" layer="1"/>
+<wire x1="6.3246" y1="27.78125" x2="6.6421" y2="27.78125" width="0.1524" layer="1"/>
 </signal>
 <signal name="INVERTED_VID_SWITCH_OUT">
@@
 <wire x1="13.391028125" y1="17.042278125" x2="12.54125" y2="17.30375" width="0.4064" layer="1" curve="-20"/>
 <wire x1="11.4554" y1="18.811875" x2="10.95375" y2="19.313525" width="0.1524" layer="1"/>
-<wire x1="11.4554" y1="18.811875" x2="11.93165" y2="19.288125" width="0.1524" layer="1"/>
+<wire x1="11.7205125" y1="19.0769875" x2="11.93165" y2="19.288125" width="0.1524" layer="1"/>
+<wire x1="11.4554" y1="18.811875" x2="11.7205125" y2="19.0769875" width="0.1524" layer="1"/>
 </signal>
 <signal name="SUB_OUT">
@@
 <wire x1="8.9154" y1="28.575" x2="8.9154" y2="27.8698" width="0.8" layer="1"/>
 <via x="8.9154" y="28.575" extent="1-16" drill="0.4" diameter="0.8"/>
-<wire x1="0" y1="20.32" x2="3.175" y2="20.32" width="1.27" layer="16"/>
+<wire x1="0" y1="20.32" x2="1.5875" y2="20.32" width="1.27" layer="16"/>
 <via x="10.795" y="48.26" extent="1-16" drill="0.4" diameter="0.8"/>
 <via x="12.7" y="48.26" extent="1-16" drill="0.4" diameter="0.8"/>
@@
 </polygon>
 </signal>
-<signal name="N$11">
+<signal name="LOGO">
 <wire x1="7.315" y1="41.28" x2="7.316" y2="41.28" width="0.3048" layer="1"/>
 <wire x1="7.815" y1="41.28" x2="7.816" y2="41.28" width="0.3048" layer="1"/>
-<wire x1="7.315" y1="41.28" x2="7.815" y2="41.28" width="0" layer="19" extent="1-1"/>
-</signal>
-<signal name="N$16">
 <wire x1="6.815" y1="41.28" x2="6.69" y2="40.78" width="0.3048" layer="1"/>
 <wire x1="6.69" y1="40.78" x2="6.815" y2="40.78" width="0.3048" layer="1"/>
@@
 <wire x1="6.315" y1="40.78" x2="6.69" y2="40.78" width="0.3048" layer="1"/>
 <wire x1="6.69" y1="40.78" x2="6.815" y2="40.78" width="0.3048" layer="1"/>
-</signal>
-<signal name="N$18">
+<wire x1="8.815" y1="41.28" x2="8.815" y2="39.28" width="0.3048" layer="1"/>
+<wire x1="8.815" y1="39.28" x2="10.815" y2="39.28" width="0.3048" layer="1"/>
+<wire x1="10.815" y1="39.28" x2="10.815" y2="41.28" width="0.3048" layer="1"/>
+<wire x1="10.815" y1="41.28" x2="8.815" y2="41.28" width="0.3048" layer="1"/>
 <wire x1="4.815" y1="41.28" x2="4.815" y2="39.78" width="0.3048" layer="1"/>
 <wire x1="4.815" y1="39.78" x2="5.315" y2="39.28" width="0.3048" layer="1" curve="90"/>
@@
 <wire x1="5.815" y1="40.78" x2="5.815" y2="40.53" width="0.3048" layer="1"/>
 <wire x1="5.815" y1="40.53" x2="5.315" y2="40.03" width="0.3048" layer="1" curve="-90"/>
-<wire x1="4.815" y1="41.28" x2="4.315" y2="40.78" width="0" layer="19" extent="1-1"/>
-</signal>
-<signal name="N$17">
-<wire x1="8.815" y1="41.28" x2="8.815" y2="39.28" width="0.3048" layer="1"/>
-<wire x1="8.815" y1="39.28" x2="10.815" y2="39.28" width="0.3048" layer="1"/>
-<wire x1="10.815" y1="39.28" x2="10.815" y2="41.28" width="0.3048" layer="1"/>
-<wire x1="10.815" y1="41.28" x2="8.815" y2="41.28" width="0.3048" layer="1"/>
-</signal>
-<signal name="N$23">
 <wire x1="9.815" y1="40.78" x2="9.315" y2="40.78" width="0.3048" layer="1"/>
 <wire x1="9.315" y1="40.78" x2="9.315" y2="40.28" width="0.3048" layer="1"/>
@@
 <wire x1="9.815" y1="39.78" x2="10.315" y2="39.78" width="0.3048" layer="1"/>
 <wire x1="10.315" y1="39.78" x2="10.315" y2="40.28" width="0.3048" layer="1"/>
-</signal>
-<signal name="N$14">
-<via x="15.24" y="35.56" extent="1-16" drill="1" diameter="2"/>
+<wire x1="7.315" y1="41.28" x2="7.815" y2="41.28" width="0" layer="19" extent="1-1"/>
+<wire x1="6.315" y1="40.78" x2="7.315" y2="41.28" width="0" layer="19" extent="1-1"/>
+<wire x1="5.815" y1="39.28" x2="6.315" y2="39.28" width="0" layer="19" extent="1-1"/>
+<wire x1="4.315" y1="40.78" x2="4.815" y2="41.28" width="0" layer="19" extent="1-1"/>
+<wire x1="9.815" y1="40.78" x2="7.815" y2="41.28" width="0" layer="19" extent="1-1"/>
 </signal>
 <signal name="AVOID1">
@@
 <vertex x="3.175" y="23.495"/>
 <vertex x="3.175" y="21.588540625"/>
-<vertex x="2.223959375" y="20.6375"/>
-<vertex x="2.223959375" y="20.0025"/>
+<vertex x="2.54" y="20.955"/>
+<vertex x="1.27" y="20.955"/>
+<vertex x="1.27" y="19.685584375"/>
+<vertex x="2.539709375" y="19.68675"/>
 <vertex x="3.175" y="19.051459375"/>
 <vertex x="3.175" y="17.145"/>
@@
 <mfgpreviewcolor name="substratecolor" color="0xFF786E46"/>
 </mfgpreviewcolors>
+<errors>
+</errors>
 </board>
 </drawing>
